Commit message: Dimention and colour changes.

File: turtle_brick/urdf/turtle.urdf.xacro (robot description, xacro)
@@ -2,17 +2,18 @@
   <!-- Define properties for the link -->
   <!-- Configured properties -->
-  <xacro:property name="platform_ground_height" value="10.0" />
-  <xacro:property name="wheel_radius" value="1.50" />
+  <xacro:property name="platform_ground_height" value="1.80" />
+  <xacro:property name="wheel_radius" value="0.30" />
   <xacro:property name="max_velocity" value="1.0" />
   <xacro:property name="gravity_accel" value="1.0" />
   <!-- Calculated properties -->
   <xacro:property name="platform_height" value="${(platform_ground_height - 2*wheel_radius) * 0.06}" />
-  <xacro:property name="cylinder_height" value="${(platform_ground_height - 2*wheel_radius) * 0.5}" />
-  <xacro:property name="base_block_height" value="${(platform_ground_height - 2*wheel_radius) * 0.3}" />
+  <xacro:property name="cylinder_height" value="${(platform_ground_height - 2*wheel_radius) * 0.42}" />
+  <xacro:property name="base_block_height" value="${(platform_ground_height - 2*wheel_radius) * 0.38}" />
   <xacro:property name="stem_height" value="${(platform_ground_height - 2*wheel_radius) * 0.1}" />
   <!-- Fixed properties -->
-  <xacro:property name="platform_radius" value="3.0" />
-  <xacro:property name="cylinder_radius" value="0.30" />
-  <xacro:property name="stem_radius" value="0.40" />
+  <xacro:property name="platform_radius" value="0.50" />
+  <xacro:property name="cylinder_radius" value="0.04" />
+  <xacro:property name="stem_radius" value="0.06" />
+  <xacro:property name="wheel_thickness" value="0.10" />
   <link name="platform">
     <visual>
@@ -21,6 +22,6 @@
         <cylinder radius = "${platform_radius}" length = "${platform_height}" />
       </geometry>
-      <material name="Green">
-        <color rgba="0 1.0 0 1.0"/>
+      <material name="Pastel orange">
+        <color rgba="0 1.0 1.0 1.0"/>
       </material>
     </visual>
@@ -32,6 +33,6 @@
         <cylinder radius = "${cylinder_radius}" length = "${cylinder_height}" />
       </geometry>
-      <material name="Green">
-        <color rgba="0 1.0 0 1.0"/>
+      <material name="Dark Green">
+        <color rgba="0.063 0.349 0.086 1.0"/>
       </material>
     </visual>
@@ -43,6 +44,6 @@
         <box size="${base_block_height} ${base_block_height} ${base_block_height}" />
       </geometry>
-      <material name="Cyan">
-        <color rgba="0 1.0 1.0 1.0"/>
+      <material name="Greenish">
+        <color rgba="0.58 0.651 0.235 1.0"/>
       </material>
     </visual>
@@ -54,6 +55,6 @@
         <cylinder radius = "${stem_radius}" length = "${stem_height}" />
       </geometry>
-      <material name="Red">
-        <color rgba="1.0 0 0 1.0"/>
+      <material name="Cobalt">
+        <color rgba="0.047 0.31 0.588 1.0"/>
       </material>
     </visual>
@@ -63,5 +64,5 @@
       <origin xyz="0 0 0" rpy="0 1.57 0" />
       <geometry>
-        <cylinder radius = "${wheel_radius}" length = "0.5" />
+        <cylinder radius = "${wheel_radius}" length = "${wheel_thickness}" />
       </geometry>
       <material name="Black">
